Commit message: prefix

File: ur5_description/urdf/ur5.urdf.xacro (robot description, xacro)
@@ -307,5 +307,5 @@
       <child link="${prefix}tool0"/>
     </joint>
-    <link name="support">
+    <link name="${prefix}support">
         <visual>
             <geometry>
@@ -324,13 +324,13 @@
         </collision>
     </link>
-    <joint name="support2wrist_3_link" type="fixed">
+    <joint  name="${prefix}support2wrist_3_link" type="fixed">
         <parent link="${prefix}wrist_3_link" />
-        <child link="support" />
+        <child link="${prefix}support" />
         <origin xyz="0 0.05 0.05" />
     </joint>
-    <gazebo reference="support">
+    <gazebo reference="${prefix}support">
         <material>Gazebo/White</material>
     </gazebo>
-	<xacro:realsense_d435 sensor_name="d435" parent_link="support" rate="10">
+	<xacro:realsense_d435 sensor_name="${prefix}d435" parent_link="${prefix}support" rate="10">
     <origin rpy="0 0 1.57 " xyz="0 0 0.01"/>
     </xacro:realsense_d435>

Commit message: disable d435

File: ur5_description/urdf/ur5.urdf.xacro (robot description, xacro)
@@ -69,5 +69,5 @@
     </inertial>
   </xacro:macro>
-  <xacro:macro name="ur5_robot" params="prefix joint_limited">
+  <xacro:macro name="ur5_robot" params="prefix joint_limited enable_d435">
     <link name="${prefix}base_link" >
       <visual>
@@ -332,7 +332,9 @@
         <material>Gazebo/White</material>
     </gazebo>
-	<xacro:realsense_d435 sensor_name="${prefix}d435" parent_link="${prefix}support" rate="10">
-    <origin rpy="0 0 1.57 " xyz="0 0 0.01"/>
-    </xacro:realsense_d435>
+    <xacro:if value="${enable_d435}">
+      <xacro:realsense_d435 sensor_name="${prefix}d435" parent_link="${prefix}support" rate="10">
+        <origin rpy="0 0 1.57 " xyz="0 0 0.01"/>
+      </xacro:realsense_d435>
+    </xacro:if>
   </xacro:macro>
 </robot>
